Commit message: Add effort-controlled gripper action bridge
Co-authored-by: Copilot <223556219+Copilot@users.noreply.github.com>

File: ros2_ws/src/robotiq_description/urdf/2f_85.ros2_control.xacro (robot description, xacro)
@@ -15,5 +15,5 @@
         gripper_max_speed:=0.150
         gripper_max_force:=235.0
-        gripper_closed_position:=0.7929">
+        gripper_closed_position:=0.0424">
         <ros2_control name="${name}" type="system">
             <!-- Plugins -->
@@ -46,5 +46,5 @@
             </hardware>
             <!-- Joint interfaces -->
-            <!-- With Ignition or Hardware, they handle mimic joints, so we only need this command interface activated -->
+            <!-- The simplified model uses equal positive travel for both jaws. -->
             <joint name="${prefix}robotiq_85_left_knuckle_joint">
                 <command_interface name="position" />
@@ -57,40 +57,4 @@
             <xacro:if value="${use_fake_hardware or sim_isaac or sim_ignition}">
                 <joint name="${prefix}robotiq_85_right_knuckle_joint">
-                    <param name="mimic">${prefix}robotiq_85_left_knuckle_joint</param>
-                    <param name="multiplier">-1</param>
-                    <xacro:unless value="${sim_ignition}">
-                        <command_interface name="position"/>
-                        <state_interface name="position"/>
-                        <state_interface name="velocity"/>
-                    </xacro:unless>
-                </joint>
-                <joint name="${prefix}robotiq_85_left_inner_knuckle_joint">
-                    <param name="mimic">${prefix}robotiq_85_left_knuckle_joint</param>
-                    <param name="multiplier">1</param>
-                    <xacro:unless value="${sim_ignition}">
-                        <command_interface name="position"/>
-                        <state_interface name="position"/>
-                        <state_interface name="velocity"/>
-                    </xacro:unless>
-                </joint>
-                <joint name="${prefix}robotiq_85_right_inner_knuckle_joint">
-                    <param name="mimic">${prefix}robotiq_85_left_knuckle_joint</param>
-                    <param name="multiplier">-1</param>
-                    <xacro:unless value="${sim_ignition}">
-                        <command_interface name="position"/>
-                        <state_interface name="position"/>
-                        <state_interface name="velocity"/>
-                    </xacro:unless>
-                </joint>
-                <joint name="${prefix}robotiq_85_left_finger_tip_joint">
-                    <param name="mimic">${prefix}robotiq_85_left_knuckle_joint</param>
-                    <param name="multiplier">-1</param>
-                    <xacro:unless value="${sim_ignition}">
-                        <command_interface name="position"/>
-                        <state_interface name="position"/>
-                        <state_interface name="velocity"/>
-                    </xacro:unless>
-                </joint>
-                <joint name="${prefix}robotiq_85_right_finger_tip_joint">
                     <param name="mimic">${prefix}robotiq_85_left_knuckle_joint</param>
                     <param name="multiplier">1</param>

File: ros2_ws/src/robotiq_description/urdf/robotiq_2f_85_macro.urdf.xacro (robot description, xacro)
@@ -18,6 +18,7 @@
         gripper_max_speed:=0.150
         gripper_max_force:=235.0
-        gripper_closed_position:=0.7929
-        use_urdf_mimic:=true">
+        gripper_closed_position:=0.0424
+        joint_effort_limit:=40.0
+        finger_travel:=0.0424">
         <!-- ros2 control include -->
         <xacro:include filename="$(find robotiq_description)/urdf/2f_85.ros2_control.xacro" />
@@ -125,14 +126,4 @@
         </link>
         <link name="${prefix}robotiq_85_left_inner_knuckle_link">
-            <visual>
-                <geometry>
-                    <mesh filename="package://robotiq_description/meshes/visual/2f_85/left_inner_knuckle.dae" />
-                </geometry>
-            </visual>
-            <collision>
-                <geometry>
-                    <mesh filename="package://robotiq_description/meshes/collision/2f_85/left_inner_knuckle.stl" />
-                </geometry>
-            </collision>
             <inertial>
                 <origin xyz="0.01897699 0.00015001 0.02247101" rpy="0 0 0" />
@@ -142,14 +133,4 @@
         </link>
         <link name="${prefix}robotiq_85_right_inner_knuckle_link">
-            <visual>
-                <geometry>
-                    <mesh filename="package://robotiq_description/meshes/visual/2f_85/right_inner_knuckle.dae" />
-                </geometry>
-            </visual>
-            <collision>
-                <geometry>
-                    <mesh filename="package://robotiq_description/meshes/collision/2f_85/right_inner_knuckle.stl" />
-                </geometry>
-            </collision>
             <inertial>
                 <origin xyz="-0.01926824 5.001e-05 0.02222178" rpy="0 0 0" />
@@ -171,6 +152,6 @@
                     <friction>
                     <ode>
-                        <mu1>100000.0</mu1>
-                        <mu2>100000.0</mu2>
+                        <mu>2.0</mu>
+                        <mu2>2.0</mu2>
                     </ode>
                     </friction>
@@ -206,6 +187,6 @@
                     <friction>
                     <ode>
-                        <mu1>100000.0</mu1>
-                        <mu2>100000.0</mu2>
+                        <mu>2.0</mu>
+                        <mu2>2.0</mu2>
                     </ode>
                     </friction>
@@ -233,20 +214,17 @@
             <xacro:insert_block name="origin" />
         </joint>
-        <joint name="${prefix}robotiq_85_left_knuckle_joint" type="revolute">
+        <joint name="${prefix}robotiq_85_left_knuckle_joint" type="prismatic">
             <parent link="${prefix}robotiq_85_base_link" />
             <child link="${prefix}robotiq_85_left_knuckle_link" />
-            <axis xyz="0 -1 0" />
+            <axis xyz="-1 0 0" />
             <origin xyz="0.03060114 0.0 0.05490452" rpy="0 0 0" />
-            <limit lower="0.0" upper="0.8" velocity="0.5" effort="50" />
-        </joint>
-        <joint name="${prefix}robotiq_85_right_knuckle_joint" type="revolute">
+            <limit lower="0.0" upper="${finger_travel}" velocity="0.05" effort="${joint_effort_limit}" />
+        </joint>
+        <joint name="${prefix}robotiq_85_right_knuckle_joint" type="prismatic">
             <parent link="${prefix}robotiq_85_base_link" />
             <child link="${prefix}robotiq_85_right_knuckle_link" />
-            <axis xyz="0 -1 0" />
+            <axis xyz="1 0 0" />
             <origin xyz="-0.03060114 0.0 0.05490452" rpy="0 0 0" />
-            <limit lower="-0.8" upper="0.0" velocity="0.5" effort="50" />
-            <xacro:if value="${use_urdf_mimic}">
-                <mimic joint="${prefix}robotiq_85_left_knuckle_joint" multiplier="-1" />
-            </xacro:if>
+            <limit lower="0.0" upper="${finger_travel}" velocity="0.05" effort="${joint_effort_limit}" />
         </joint>
         <joint name="${prefix}robotiq_85_left_finger_joint" type="fixed">
@@ -260,43 +238,23 @@
             <origin xyz="-0.03152616 0.0 -0.00376347" rpy="0 0 0" />
         </joint>
-        <joint name="${prefix}robotiq_85_left_inner_knuckle_joint" type="revolute">
+        <joint name="${prefix}robotiq_85_left_inner_knuckle_joint" type="fixed">
             <parent link="${prefix}robotiq_85_base_link" />
             <child link="${prefix}robotiq_85_left_inner_knuckle_link" />
-            <axis xyz="0 -1 0" />
             <origin xyz="0.0127 0.0 0.06142" rpy="0 0 0" />
-            <xacro:if value="${use_urdf_mimic}">
-                <mimic joint="${prefix}robotiq_85_left_knuckle_joint" />
-            </xacro:if>
-            <limit lower="0.0" upper="0.8" velocity="0.5" effort="50" />
-        </joint>
-        <joint name="${prefix}robotiq_85_right_inner_knuckle_joint" type="revolute">
+        </joint>
+        <joint name="${prefix}robotiq_85_right_inner_knuckle_joint" type="fixed">
             <parent link="${prefix}robotiq_85_base_link" />
             <child link="${prefix}robotiq_85_right_inner_knuckle_link" />
-            <axis xyz="0 -1 0" />
             <origin xyz="-0.0127 0.0 0.06142" rpy="0 0 0" />
-            <xacro:if value="${use_urdf_mimic}">
-                <mimic joint="${prefix}robotiq_85_left_knuckle_joint" multiplier="-1" />
-            </xacro:if>
-            <limit lower="-0.8" upper="0.0" velocity="0.5" effort="50" />
-        </joint>
-        <joint name="${prefix}robotiq_85_left_finger_tip_joint" type="revolute">
+        </joint>
+        <joint name="${prefix}robotiq_85_left_finger_tip_joint" type="fixed">
             <parent link="${prefix}robotiq_85_left_finger_link" />
             <child link="${prefix}robotiq_85_left_finger_tip_link" />
-            <axis xyz="0 -1 0" />
             <origin xyz="0.00563134 0.0 0.04718515" rpy="0 0 0" />
-            <xacro:if value="${use_urdf_mimic}">
-                <mimic joint="${prefix}robotiq_85_left_knuckle_joint" multiplier="-1" />
-            </xacro:if>
-            <limit lower="-0.8" upper="0.0" velocity="0.5" effort="50" />
-        </joint>
-        <joint name="${prefix}robotiq_85_right_finger_tip_joint" type="revolute">
+        </joint>
+        <joint name="${prefix}robotiq_85_right_finger_tip_joint" type="fixed">
             <parent link="${prefix}robotiq_85_right_finger_link" />
             <child link="${prefix}robotiq_85_right_finger_tip_link" />
-            <axis xyz="0 -1 0" />
             <origin xyz="-0.00563134 0.0 0.04718515" rpy="0 0 0" />
-            <xacro:if value="${use_urdf_mimic}">
-                <mimic joint="${prefix}robotiq_85_left_knuckle_joint" />
-            </xacro:if>
-            <limit lower="0.0" upper="0.8" velocity="0.5" effort="50" />
         </joint>
     </xacro:macro>

File: ros2_ws/src/sensoragent_rm65_b_bringup/urdf/rm65_b_robotiq_2f85.urdf.xacro (robot description, xacro)
@@ -3,5 +3,4 @@
   <xacro:arg name="gripper_mount_xyz" default="0 0 0"/>
   <xacro:arg name="gripper_mount_rpy" default="0 0 0"/>
-  <xacro:arg name="use_urdf_mimic" default="true"/>
   <link name="world"/>
   <joint name="world_to_rm65_b" type="fixed">
@@ -16,5 +15,6 @@
     parent="Link6"
     include_ros2_control="false"
-    use_urdf_mimic="$(arg use_urdf_mimic)">
+    joint_effort_limit="40.0"
+    finger_travel="0.0424">
     <origin xyz="$(arg gripper_mount_xyz)" rpy="$(arg gripper_mount_rpy)"/>
   </xacro:robotiq_gripper>
@@ -111,29 +111,18 @@
     </joint>
     <joint name="robotiq_85_left_knuckle_joint">
-      <command_interface name="position"/>
+      <command_interface name="effort"/>
       <state_interface name="position">
         <param name="initial_value">0</param>
       </state_interface>
       <state_interface name="velocity"/>
+      <state_interface name="effort"/>
     </joint>
     <joint name="robotiq_85_right_knuckle_joint">
-      <param name="mimic">robotiq_85_left_knuckle_joint</param>
-      <param name="multiplier">-1</param>
-    </joint>
-    <joint name="robotiq_85_left_inner_knuckle_joint">
-      <param name="mimic">robotiq_85_left_knuckle_joint</param>
-      <param name="multiplier">1</param>
-    </joint>
-    <joint name="robotiq_85_right_inner_knuckle_joint">
-      <param name="mimic">robotiq_85_left_knuckle_joint</param>
-      <param name="multiplier">-1</param>
-    </joint>
-    <joint name="robotiq_85_left_finger_tip_joint">
-      <param name="mimic">robotiq_85_left_knuckle_joint</param>
-      <param name="multiplier">-1</param>
-    </joint>
-    <joint name="robotiq_85_right_finger_tip_joint">
-      <param name="mimic">robotiq_85_left_knuckle_joint</param>
-      <param name="multiplier">1</param>
+      <command_interface name="effort"/>
+      <state_interface name="position">
+        <param name="initial_value">0</param>
+      </state_interface>
+      <state_interface name="velocity"/>
+      <state_interface name="effort"/>
     </joint>
   </ros2_control>
