Commit message: Stabilize RM65-B gripper simulation
Co-authored-by: Copilot <223556219+Copilot@users.noreply.github.com>

File: ros2_ws/src/robotiq_description/urdf/robotiq_2f_85_macro.urdf.xacro (robot description, xacro)
@@ -18,5 +18,6 @@
         gripper_max_speed:=0.150
         gripper_max_force:=235.0
-        gripper_closed_position:=0.7929">
+        gripper_closed_position:=0.7929
+        use_urdf_mimic:=true">
         <!-- ros2 control include -->
         <xacro:include filename="$(find robotiq_description)/urdf/2f_85.ros2_control.xacro" />
@@ -245,5 +246,7 @@
             <origin xyz="-0.03060114 0.0 0.05490452" rpy="0 0 0" />
             <limit lower="-0.8" upper="0.0" velocity="0.5" effort="50" />
-            <mimic joint="${prefix}robotiq_85_left_knuckle_joint" multiplier="-1" />
+            <xacro:if value="${use_urdf_mimic}">
+                <mimic joint="${prefix}robotiq_85_left_knuckle_joint" multiplier="-1" />
+            </xacro:if>
         </joint>
         <joint name="${prefix}robotiq_85_left_finger_joint" type="fixed">
@@ -262,5 +265,7 @@
             <axis xyz="0 -1 0" />
             <origin xyz="0.0127 0.0 0.06142" rpy="0 0 0" />
-            <mimic joint="${prefix}robotiq_85_left_knuckle_joint" />
+            <xacro:if value="${use_urdf_mimic}">
+                <mimic joint="${prefix}robotiq_85_left_knuckle_joint" />
+            </xacro:if>
             <limit lower="0.0" upper="0.8" velocity="0.5" effort="50" />
         </joint>
@@ -270,5 +275,7 @@
             <axis xyz="0 -1 0" />
             <origin xyz="-0.0127 0.0 0.06142" rpy="0 0 0" />
-            <mimic joint="${prefix}robotiq_85_left_knuckle_joint" multiplier="-1" />
+            <xacro:if value="${use_urdf_mimic}">
+                <mimic joint="${prefix}robotiq_85_left_knuckle_joint" multiplier="-1" />
+            </xacro:if>
             <limit lower="-0.8" upper="0.0" velocity="0.5" effort="50" />
         </joint>
@@ -278,5 +285,7 @@
             <axis xyz="0 -1 0" />
             <origin xyz="0.00563134 0.0 0.04718515" rpy="0 0 0" />
-            <mimic joint="${prefix}robotiq_85_left_knuckle_joint" multiplier="-1" />
+            <xacro:if value="${use_urdf_mimic}">
+                <mimic joint="${prefix}robotiq_85_left_knuckle_joint" multiplier="-1" />
+            </xacro:if>
             <limit lower="-0.8" upper="0.0" velocity="0.5" effort="50" />
         </joint>
@@ -286,5 +295,7 @@
             <axis xyz="0 -1 0" />
             <origin xyz="-0.00563134 0.0 0.04718515" rpy="0 0 0" />
-            <mimic joint="${prefix}robotiq_85_left_knuckle_joint" />
+            <xacro:if value="${use_urdf_mimic}">
+                <mimic joint="${prefix}robotiq_85_left_knuckle_joint" />
+            </xacro:if>
             <limit lower="0.0" upper="0.8" velocity="0.5" effort="50" />
         </joint>

File: ros2_ws/src/sensoragent_rm65_b_bringup/urdf/rm65_b_robotiq_2f85.urdf.xacro (robot description, xacro)
@@ -3,4 +3,5 @@
   <xacro:arg name="gripper_mount_xyz" default="0 0 0"/>
   <xacro:arg name="gripper_mount_rpy" default="0 0 0"/>
+  <xacro:arg name="use_urdf_mimic" default="true"/>
   <link name="world"/>
   <joint name="world_to_rm65_b" type="fixed">
@@ -8,5 +9,5 @@
     <child link="base_link"/>
   </joint>
-  <xacro:include filename="$(find rm_description)/urdf/rm_65_gazebo.urdf"/>
+  <xacro:include filename="$(find rm_description)/urdf/rm_65.urdf"/>
   <xacro:include filename="$(find robotiq_description)/urdf/robotiq_2f_85_macro.urdf.xacro"/>
   <xacro:robotiq_gripper
@@ -14,5 +15,6 @@
     prefix=""
     parent="Link6"
-    include_ros2_control="false">
+    include_ros2_control="false"
+    use_urdf_mimic="$(arg use_urdf_mimic)">
     <origin xyz="$(arg gripper_mount_xyz)" rpy="$(arg gripper_mount_rpy)"/>
   </xacro:robotiq_gripper>
@@ -46,4 +48,20 @@
     <gravity>false</gravity>
   </gazebo>
+  <!-- Keep the attached gripper stable before ros2_control activates. -->
+  <xacro:macro name="gazebo_gripper_link" params="link">
+    <gazebo reference="${link}">
+      <self_collide>false</self_collide>
+      <gravity>false</gravity>
+    </gazebo>
+  </xacro:macro>
+  <xacro:gazebo_gripper_link link="robotiq_85_base_link"/>
+  <xacro:gazebo_gripper_link link="robotiq_85_left_knuckle_link"/>
+  <xacro:gazebo_gripper_link link="robotiq_85_right_knuckle_link"/>
+  <xacro:gazebo_gripper_link link="robotiq_85_left_finger_link"/>
+  <xacro:gazebo_gripper_link link="robotiq_85_right_finger_link"/>
+  <xacro:gazebo_gripper_link link="robotiq_85_left_inner_knuckle_link"/>
+  <xacro:gazebo_gripper_link link="robotiq_85_right_inner_knuckle_link"/>
+  <xacro:gazebo_gripper_link link="robotiq_85_left_finger_tip_link"/>
+  <xacro:gazebo_gripper_link link="robotiq_85_right_finger_tip_link"/>
   <ros2_control name="RM65BWithRobotiqSystem" type="system">
     <hardware>
@@ -121,5 +139,5 @@
   </ros2_control>
   <gazebo>
-    <self_collide>true</self_collide>
+    <self_collide>false</self_collide>
     <plugin filename="gz_ros2_control-system" name="gz_ros2_control::GazeboSimROS2ControlPlugin">
       <parameters>$(find sensoragent_rm65_b_bringup)/config/ros2_controllers.yaml</parameters>

Commit message: Improve Gazebo pick and place reliability
Co-authored-by: Copilot <223556219+Copilot@users.noreply.github.com>

File: ros2_ws/src/robotiq_description/urdf/robotiq_2f_85_macro.urdf.xacro (robot description, xacro)
@@ -79,4 +79,12 @@
                     <mesh filename="package://robotiq_description/meshes/collision/2f_85/left_finger.stl" />
                 </geometry>
+                <surface>
+                    <friction>
+                        <ode>
+                            <mu>5.0</mu>
+                            <mu2>5.0</mu2>
+                        </ode>
+                    </friction>
+                </surface>
             </collision>
             <visual name="finger_tip_visual">
@@ -94,6 +102,6 @@
                     <friction>
                         <ode>
-                            <mu>2.0</mu>
-                            <mu2>2.0</mu2>
+                            <mu>5.0</mu>
+                            <mu2>5.0</mu2>
                         </ode>
                     </friction>
@@ -144,4 +152,12 @@
                     <mesh filename="package://robotiq_description/meshes/collision/2f_85/right_finger.stl" />
                 </geometry>
+                <surface>
+                    <friction>
+                        <ode>
+                            <mu>5.0</mu>
+                            <mu2>5.0</mu2>
+                        </ode>
+                    </friction>
+                </surface>
             </collision>
             <visual name="finger_tip_visual">
@@ -159,6 +175,6 @@
                     <friction>
                         <ode>
-                            <mu>2.0</mu>
-                            <mu2>2.0</mu2>
+                            <mu>5.0</mu>
+                            <mu2>5.0</mu2>
                         </ode>
                     </friction>

File: ros2_ws/src/sensoragent_rm65_b_bringup/urdf/rm65_b_robotiq_2f85.urdf.xacro (robot description, xacro)
@@ -3,4 +3,6 @@
   <xacro:arg name="gripper_mount_xyz" default="0 0 0"/>
   <xacro:arg name="gripper_mount_rpy" default="0 0 0"/>
+  <xacro:arg name="gripper_tcp_xyz" default="0 0 0.10"/>
+  <xacro:arg name="gripper_tcp_rpy" default="0 0 0"/>
   <xacro:arg name="robot_mount_xyz" default="0 0 0.18"/>
   <xacro:arg name="robot_mount_rpy" default="0 0 0"/>
@@ -22,4 +24,10 @@
     <origin xyz="$(arg gripper_mount_xyz)" rpy="$(arg gripper_mount_rpy)"/>
   </xacro:robotiq_gripper>
+  <link name="robotiq_85_tcp"/>
+  <joint name="robotiq_85_tcp_joint" type="fixed">
+    <origin xyz="$(arg gripper_tcp_xyz)" rpy="$(arg gripper_tcp_rpy)"/>
+    <parent link="robotiq_85_base_link"/>
+    <child link="robotiq_85_tcp"/>
+  </joint>
   <gazebo reference="base_link">
     <self_collide>false</self_collide>
