Commit message: model refine

File: ros2_ws/src/sensoragent_rm65_b_bringup/urdf/rm65_b_robotiq_2f85.urdf.xacro (robot description, xacro)
@@ -3,6 +3,9 @@
   <xacro:arg name="gripper_mount_xyz" default="0 0 0"/>
   <xacro:arg name="gripper_mount_rpy" default="0 0 0"/>
+  <xacro:arg name="robot_mount_xyz" default="0 0 0.30"/>
+  <xacro:arg name="robot_mount_rpy" default="0 0 0"/>
   <link name="world"/>
   <joint name="world_to_rm65_b" type="fixed">
+    <origin xyz="$(arg robot_mount_xyz)" rpy="$(arg robot_mount_rpy)"/>
     <parent link="world"/>
     <child link="base_link"/>
